File: pcb/net-stepper2.sch (EAGLE design)
At the start: 38 parts, among them J1 MICRO-USB, J2 POWER_JACKPTH_LOCK, J3 ENCODER, J4 ENDSTOP2, J5 ENDSTOP1, J6 STEPER, Q1 600mA/40V, Q2 600mA/40V, U1 L6470, U2 CP2104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

Commit message: Last check
Parts:
- removed R5: 8.2k, SparkFun-Passives:RESISTOR0603-RES
- added JP1: (no value), RP400N501A:JUMPER-2SMD-NC
Connections:
- net VBUS renamed N$1
- net GND: now also JP1.2; no longer R5.1
- net SC_ADC: now also JP1.1; no longer R5.2
- net SC_CSN: now also U5.25-IOD; no longer U5.5
Changed lines of the file:
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@@
 <part name="C3" library="SparkFun-Capacitors" deviceset="100UF-63V-20%(ELECT)" device="" value="100uF"/>
 <part name="P+2" library="SparkFun" deviceset="VCC" device="" value="VS"/>
-<part name="R5" library="SparkFun-Passives" deviceset="RESISTOR" device="0603-RES" value="8.2k"/>
 <part name="GND8" library="SparkFun" deviceset="GND" device=""/>
 <part name="P+5" library="SparkFun-Aesthetics" deviceset="3.3V" device=""/>
@@
 <part name="U$33" library="microbuilder" deviceset="GND" device=""/>
 <part name="U$34" library="microbuilder" deviceset="GND" device=""/>
-<part name="U$36" library="microbuilder" deviceset="VBUS" device=""/>
 <part name="U$38" library="microbuilder" deviceset="3.3V" device=""/>
 <part name="J1" library="SparkFun-Connectors" deviceset="USB_MICRO-B" device="_SMT" value="MICRO-USB"/>
@@
 <part name="C7" library="SparkFun-Capacitors" deviceset="10UF" device="-0603-6.3V-20%" value="10uF"/>
 <part name="U$18" library="microbuilder" deviceset="GND" device=""/>
+<part name="JP1" library="RP400N501A" deviceset="JUMPER-2" device="SMD-NC"/>
 </parts>
 <sheets>
@@
 <instance part="D1" gate="G$1" x="177.8" y="127" rot="R270"/>
 <instance part="C6" gate="G$1" x="162.56" y="127" rot="R270"/>
-<instance part="C5" gate="G$1" x="190.5" y="127" smashed="yes" rot="R180">
-<attribute name="NAME" x="188.976" y="124.079" size="1.778" layer="95" rot="R180"/>
-</instance>
+<instance part="C5" gate="G$1" x="190.5" y="127" rot="R180"/>
 <instance part="C4" gate="G$1" x="48.26" y="15.24"/>
 <instance part="C3" gate="G$1" x="30.48" y="17.78"/>
 <instance part="P+2" gate="1" x="30.48" y="30.48"/>
-<instance part="R5" gate="G$1" x="175.26" y="160.02" rot="R90"/>
 <instance part="GND8" gate="1" x="175.26" y="149.86"/>
 <instance part="P+5" gate="G$1" x="149.86" y="182.88"/>
@@
 <instance part="U$33" gate="G$1" x="449.58" y="96.52"/>
 <instance part="U$34" gate="G$1" x="472.44" y="121.92"/>
-<instance part="U$36" gate="G$1" x="452.12" y="127"/>
 <instance part="U$38" gate="G$1" x="472.44" y="152.4"/>
 <instance part="J1" gate="G$1" x="439.42" y="114.3" rot="R180"/>
@@
 <instance part="C7" gate="G$1" x="462.28" y="129.54"/>
 <instance part="U$18" gate="G$1" x="462.28" y="121.92"/>
+<instance part="JP1" gate="A" x="177.8" y="157.48" rot="R270"/>
 </instances>
 <busses>
@@
 <segment>
 <wire x1="175.26" y1="154.94" x2="175.26" y2="152.4" width="0.1524" layer="91"/>
-<pinref part="R5" gate="G$1" pin="1"/>
 <pinref part="GND8" gate="1" pin="GND"/>
+<pinref part="JP1" gate="A" pin="2"/>
 </segment>
 <segment>
@@
 </segment>
 <segment>
-<wire x1="175.26" y1="165.1" x2="175.26" y2="167.64" width="0.1524" layer="91"/>
+<wire x1="175.26" y1="157.48" x2="175.26" y2="167.64" width="0.1524" layer="91"/>
 <wire x1="175.26" y1="167.64" x2="187.96" y2="167.64" width="0.1524" layer="91"/>
-<pinref part="R5" gate="G$1" pin="2"/>
 <label x="187.96" y="167.64" size="1.778" layer="95" xref="yes"/>
+<pinref part="JP1" gate="A" pin="1"/>
 </segment>
 </net>
@@
 </segment>
 <segment>
-<label x="353.06" y="129.54" size="1.27" layer="95" xref="yes"/>
-<pinref part="U5" gate="G$1" pin="5"/>
-<wire x1="345.44" y1="129.54" x2="353.06" y2="129.54" width="0.1524" layer="91"/>
+<label x="284.48" y="129.54" size="1.27" layer="95" rot="R180" xref="yes"/>
+<pinref part="U5" gate="G$1" pin="25-IOD"/>
+<wire x1="289.56" y1="129.54" x2="284.48" y2="129.54" width="0.1524" layer="91"/>
+<wire x1="292.1" y1="129.54" x2="289.56" y2="129.54" width="0.1524" layer="91"/>
 </segment>
 </net>
@@
 </segment>
 </net>
-<net name="VBUS" class="0">
-<segment>
-<wire x1="452.12" y1="116.84" x2="477.52" y2="116.84" width="0.1524" layer="91"/>
-<pinref part="U$36" gate="G$1" pin="VBUS"/>
-<wire x1="452.12" y1="116.84" x2="452.12" y2="124.46" width="0.1524" layer="91"/>
-<pinref part="J1" gate="G$1" pin="VBUS"/>
-<wire x1="444.5" y1="109.22" x2="452.12" y2="109.22" width="0.1524" layer="91"/>
-<wire x1="452.12" y1="109.22" x2="452.12" y2="116.84" width="0.1524" layer="91"/>
-<junction x="452.12" y="116.84"/>
-<pinref part="U2" gate="G$1" pin="VBUS"/>
-</segment>
-</net>
 <net name="N$13" class="0">
 <segment>
@@
 </segment>
 </net>
+<net name="N$1" class="0">
+<segment>
+<wire x1="452.12" y1="116.84" x2="477.52" y2="116.84" width="0.1524" layer="91"/>
+<pinref part="J1" gate="G$1" pin="VBUS"/>
+<wire x1="444.5" y1="109.22" x2="452.12" y2="109.22" width="0.1524" layer="91"/>
+<wire x1="452.12" y1="109.22" x2="452.12" y2="116.84" width="0.1524" layer="91"/>
+<pinref part="U2" gate="G$1" pin="VBUS"/>
+</segment>
+</net>

Commit message: added todo
Other:
- note added: "FIX: External power requirement to flash the device. Actually, the esp32 is powered somehow through the usb bridge..."
Changed lines of the file:
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@@
 <text x="474.98" y="157.48" size="1.778" layer="94">USB TO SERIAL CONVERTER</text>
 <text x="205.74" y="25.4" size="1.778" layer="94">RGB LED</text>
+<text x="149.86" y="210.82" size="5.08" layer="94">FIX: External power requirement to flash the device. Actually, the esp32 is powered somehow through the usb bridge...</text>
 </plain>
 <instances>
